File: EspressoMachineBoard/EspressoMachineBoard.kicad_pcb (KiCad board)
At the start: 2 copper layers, 130 x 60 mm, 71 parts, among them J2 54132-4062, K1 G2RL-1A-E-HA DC5, K2 G2RL-1A-E-HA DC5, Q1 BTA16-600B, Q4 BTA16-600B, U1 ESP32-S3-WROOM-2, U2 AP7361C-33E, U3 LTV-354T, U4 FOD420, U6 FOD420, U8 LM4041LP-ADJ, U9 LM358_DFN

Commit message: Boards finalized and ordered
Parts:
- removed K1, K2: G2RL-1A-E-HA DC5, Relay_THT:Relay_SPST_Omron_G2RL-1A-E
- removed PS1: TMLM04105, Converter_ACDC:Converter_ACDC_TRACO_TMLM-04_THT
- removed Q4: BTA16-600B, Package_TO_SOT_THT:TO-220-3_Vertical
- removed R10, R14, R18: 10k, Resistor_SMD:R_0603_1608Metric_Pad0.98x0.95mm_HandSolder
- removed R11, R15: 65, Resistor_SMD:R_0603_1608Metric_Pad0.98x0.95mm_HandSolder
- removed R12, R13: 1k, Resistor_SMD:R_0603_1608Metric_Pad0.98x0.95mm_HandSolder
- removed R21, R22, R25, R26, R27: R, Resistor_SMD:R_0603_1608Metric_Pad0.98x0.95mm_HandSolder
- removed TP10, TP11, TP12, TP13, TP14, TP20, TP21, TP23, TP24, TP25, TP4, TP5, TP6, TP7, TP9: TestPoint, Connector_PinHeader_2.54mm:PinHeader_1x01_P2.54mm_Vertical
- removed U4: FOD420, Package_DIP:DIP-6_W7.62mm
- removed U8: LM4041LP-ADJ, Package_TO_SOT_THT:TO-92_Inline
- added BZ1: Buzzer, Buzzer_Beeper:Buzzer_TDK_PS1240P02BT_D12.2mm_H6.5mm, B.Cu at (84.0, 64.5)
- added C1: 100n, Capacitor_SMD:C_0603_1608Metric_Pad1.08x0.95mm_HandSolder, F.Cu at (86.9, 29.0)
- added C2: 100n, Capacitor_SMD:C_0603_1608Metric_Pad1.08x0.95mm_HandSolder, F.Cu at (90.0, 38.9)
- added F1: 1A, Fuse:Fuse_0603_1608Metric_Pad1.05x0.95mm_HandSolder, F.Cu at (20.4, 38.0)
- added H1: MountingHole_Pad, MountingHole:MountingHole_3.2mm_M3_DIN965, F.Cu at (25.0, 20.0)
- added H2: MountingHole_Pad, MountingHole:MountingHole_3.2mm_M3_DIN965, F.Cu at (127.0, 20.0)
- added H3: MountingHole_Pad, MountingHole:MountingHole_3.2mm_M3_DIN965, F.Cu at (25.0, 74.9)
- added H4: MountingHole_Pad, MountingHole:MountingHole_3.2mm_M3_DIN965, F.Cu at (127.0, 74.9)
- added H5: MountingHole_Pad, MountingHole:MountingHole_3.2mm_M3_DIN965_Pad, F.Cu at (16.0, 16.0)
- added H6: MountingHole_Pad, MountingHole:MountingHole_3.2mm_M3_DIN965_Pad, F.Cu at (158.0, 16.0)
- added H7: MountingHole_Pad, MountingHole:MountingHole_3.2mm_M3_DIN965_Pad, F.Cu at (16.0, 83.0)
- added H8: MountingHole_Pad, MountingHole:MountingHole_3.2mm_M3_DIN965_Pad, F.Cu at (158.0, 83.0)
- added J1: USB_C_Receptacle_USB2.0_14P, Connector_USB:USB_C_Receptacle_GCT_USB4110, B.Cu at (15.8, 26.9)
- added J3: Conn_01x02_Pin, Connector_JST:JST_XH_B2B-XH-AM_1x02_P2.50mm_Vertical, F.Cu at (98.2, 33.1)
- added J4: Conn_01x02_Pin, Connector_PinSocket_2.54mm:PinSocket_1x02_P2.54mm_Vertical, F.Cu at (80.0, 25.8)
- added J5: Conn_01x08_Pin, Connector_JST:JST_PH_B8B-PH-K_1x08_P2.00mm_Vertical, B.Cu at (39.5, 83.5)
- added J6: Conn_01x14_Pin, Connector_PinSocket_2.54mm:PinSocket_1x14_P2.54mm_Vertical, B.Cu at (128.0, 30.9)
- added J7: Conn_01x14_Pin, Connector_PinSocket_2.54mm:PinSocket_1x14_P2.54mm_Vertical, F.Cu at (124.2, 31.0)
- added JP1: Jumper_2_Open, Jumper:SolderJumper-2_P1.3mm_Open_Pad1.0x1.5mm, F.Cu at (21.5, 34.6)
- added JP2: Jumper_2_Open, Jumper:SolderJumper-2_P1.3mm_Open_Pad1.0x1.5mm, F.Cu at (22.5, 47.0)
- added JP3: Jumper_2_Open, Jumper:SolderJumper-2_P1.3mm_Open_Pad1.0x1.5mm, B.Cu at (90.8, 22.2)
- added JP4: Jumper_2_Open, Jumper:SolderJumper-2_P1.3mm_Open_Pad1.0x1.5mm, B.Cu at (90.8, 24.8)
- added Q2: NMOS, Package_TO_SOT_SMD:SOT-23, F.Cu at (83.9, 53.5)
- added Q7: NMOS, Package_TO_SOT_SMD:SOT-23, F.Cu at (119.8, 24.8)
- added Q8: NMOS, Package_TO_SOT_SMD:SOT-23, F.Cu at (130.1, 26.5)
- added Q9: NMOS, Package_TO_SOT_SMD:SOT-23, F.Cu at (118.3, 19.5)
- added R5: 37.5k, Resistor_SMD:R_0603_1608Metric_Pad0.98x0.95mm_HandSolder, F.Cu at (84.5, 38.0)
- added R6: 37.5k, Resistor_SMD:R_0603_1608Metric_Pad0.98x0.95mm_HandSolder, F.Cu at (87.0, 40.0)
- added SW1: SW_Push, Button_Switch_SMD:SW_Push_1P1T_NO_6x6mm_H9.5mm, B.Cu at (75.0, 51.2)
- added SW2: SW_Push, Button_Switch_SMD:SW_Push_1P1T_NO_6x6mm_H9.5mm, B.Cu at (36.5, 23.0)
- added SW3: RotaryEncoder_Switch, Rotary_Encoder:RotaryEncoder_Alps_EC11E-Switch_Vertical_H20mm, F.Cu at (135.0, 46.8)
- added SW4: SW_SPDT, Button_Switch_THT:SW_Slide_SPDT_Straight_CK_OS102011MS2Q, F.Cu at (140.0, 72.8)
- added U5: 74AHC1G08GW,125, Package_TO_SOT_SMD:SOT-353_SC-70-5_Handsoldering, F.Cu at (55.5, 53.5)
- J2: value 54132-4062 -> Conn_01x04_Pin; footprint EspressoMachineHW:54132-4062_1 -> Connector_PinSocket_2.54mm:PinSocket_1x04_P2.54mm_Vertical
- LED1: moved to B.Cu
- Q1: value BTA16-600B -> NMOS; footprint Package_TO_SOT_THT:TO-220-3_Vertical -> Package_TO_SOT_SMD:SOT-23
- R23, R31: value R -> 10k
- R24: value R -> 3k
- U3: value LTV-354T -> LM358_DFN; footprint Package_SO:SO-4_4.4x3.6mm_P2.54mm -> Package_SO:SOIC-8_3.9x4.9mm_P1.27mm
- U6: value FOD420 -> LM4040DCK-2.5; footprint Package_DIP:DIP-6_W7.62mm -> Package_TO_SOT_SMD:SOT-353_SC-70-5
- U9: footprint Package_DFN_QFN:DFN-8-1EP_2x2mm_P0.5mm_EP1.05x1.75mm -> Package_SO:SOIC-8_3.9x4.9mm_P1.27mm
- moved TP3 268.4 mm to (157.0, 50.2)
- moved TP18 237.5 mm to (148.5, 23.0)
- moved TP17 234.2 mm to (144.8, 23.0)
- moved TP16 205.1 mm to (114.0, 27.5)
- moved J2 189.6 mm to (99.0, 24.8), turned to 90 degrees
- moved TP8 188.0 mm to (85.5, 21.5)
- moved D3 179.5 mm to (147.3, 18.2), turned to 180 degrees
- moved R4 178.3 mm to (143.3, 18.2)
- moved R19 176.7 mm to (114.0, 23.0), turned to 90 degrees
- moved TP15 166.3 mm to (61.0, 60.5)
- moved LED1 164.4 mm to (142.0, 32.0), turned to 180 degrees
- moved R30 155.5 mm to (133.3, 18.8), turned to 180 degrees
- moved R29 155.4 mm to (133.2, 27.7), turned to 90 degrees
- moved TP2 154.1 mm to (24.5, 61.5)
- moved R28 153.9 mm to (131.8, 23.8), turned to 180 degrees
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Connections:
- J2 pad 1: GND -> /MTMS/IO42
- J2 pad 2: /DISPLAY_MOSI -> /MTDI/IO41
- J2 pad 3: +3.3V -> /MTDO/IO40
- J2 pad 4: /DISPLAY_FRMARK -> /MTCK/IO39
- Q1 pad 1: /PUMP_HOT_OUT -> Net-(J6-Pin_7)
- Q1 pad 2: /120VAC_HOT_SWITCHED -> /~{LCD_LED}
- Q1 pad 3: Net-(Q1-G) -> GND
- R31 pad 1: /STEAM_VALVE_IN -> /STEAM_VALVE_SIG
- TP2 pad 1: /DISPLAY_DC -> GND
- TP3 pad 1: /DISPLAY_CS0 -> GND
- TP8 pad 1: /DISPLAY_FRMARK -> /THERMISTOR_SIG_ANALOG
- U1 pad 10: /USR_HV_SWITCH -> /ROTARYENC_SWITCH
- U1 pad 12: /BUZZER -> /SD_CS
- U1 pad 23: /IO21 -> /~{LCD_LED}
- U1 pad 26: /BUZZER -> /STEAM_VALVE_SIG
- U1 pad 27: /THERMISTOR_SIG_ANALOG -> /BUZZER
- U1 pad 31: /IO38 -> /LCD_CTP_SDA
- U1 pad 38: /LCD_CTP_RST -> /THERMISTOR_SIG_ANALOG
- U1 pad 4: /LCD_CTP_SDA -> /LCD_CTP_RST
- U1 pad 8: /DISPLAY_FRMARK -> /USR_HV_SWITCH
- U3 pad 1: Net-(R8-Pad1) -> Net-(U3A--)
- U3 pad 2: Net-(R9-Pad1) -> Net-(U3A--)
- U3 pad 3: GND -> /THERMISTOR_OUT
- U3 pad 4: /AC_ZC -> GND
- U6 pad 1: Net-(R15-Pad2) -> GND
- U6 pad 2: Net-(Q3-D) -> unconnected-(U6-NC-Pad2)
- U6 pad 3: unconnected-(U6-NC-Pad3) -> /THERMISTOR_IN
- U6 pad 4: Net-(Q4-G) -> unconnected-(U6-NC-Pad4)
Routing:
- net GND: track 0.00 -> 243.1 mm, vias 0 -> 23
- net /USR_HV_SWITCH: track 0.00 -> 130.3 mm, vias 0 -> 2
- net +5V: track 0.00 -> 120.2 mm, vias 0 -> 1
- net /ROTARYENC_SWITCH: track 0.00 -> 114.8 mm, vias 0 -> 1
- net /STEAM_VALVE_SIG: track 0.00 -> 102.3 mm, vias 0 -> 4
- net +3.3V: track 0.00 -> 96.1 mm, vias 0 -> 17
- net /ROTARYENC_B: track 0.00 -> 94.6 mm
- net /ROTARYENC_A: track 0.00 -> 83.2 mm
- net /DISPLAY_CS0: track 0.00 -> 81.8 mm, vias 0 -> 2
- net /SD_CS: track 0.00 -> 79.0 mm, vias 0 -> 2
- net /LCD_CTP_RST: track 0.00 -> 79.0 mm, vias 0 -> 1
- net /LCD_CTP_SCL: track 0.00 -> 76.6 mm, vias 0 -> 1
- net /DISPLAY_DC: track 0.00 -> 74.9 mm
- net /BOILER_TRIAC: track 0.00 -> 73.9 mm, vias 0 -> 2
- net /PUMP_TRIAC: track 0.00 -> 72.3 mm, vias 0 -> 2
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- added copper zone on B.Cu, net +3.3V
- added copper zone on B.Cu, net GND
- added copper zone on F.Cu, net GND
Other:
- board size 130 x 60 mm -> 150 x 75 mm
- board text added: "+3.3V"
- board text added: "+5V"
- board text added: "AC Control Board Connector"
- board text added: "AC Relays"
- board text added: "AC Switch"
- board text added: "Boiler Triac Out"
- board text added: "CLK"
- board text added: "CTP_INT"
- board text added: "CTP_RST"
- board text added: "CTP_SCL"
- board text added: "CTP_SDA"
- board text added: "Debug"
- board text added: "Display"
- board text added: "ENC_A"
- board text added: "ENC_B"
- board text added: "Espresso Machine Controller Project"
- board text added: "GND"
- board text added: "JTAG"
- board text added: "Knob"
- board text added: "LCD"
- board text added: "LCD_CS"
- board text added: "LCD_DC"
- board text added: "LCD_RST"
- board text added: "LED"
- board text added: "MISO"
- board text added: "MOSI"
- board text added: "Main Control Board"
- board text added: "PWR"
- board text added: "Pres"
- board text added: "Pres. Sensor In"
- board text added: "Pump Triac Out"
- board text added: "RX"
- board text added: "Relay Out"
- board text added: "SD_CS"
- board text added: "Steam Sensor In"
- board text added: "TCK"
- board text added: "TDI"
- board text added: "TDO"
- board text added: "TMS"
- board text added: "TX"
- board text added: "Therm"
- board text added: "Thermistor"
- board text added: "Usr AC"
- board text added: "ZC In"
