File: EspressoMachineBoard/EspressoMachineBoard.kicad_sch (KiCad schematic)
At the start: 48 parts, among them J1 USB_C_Receptacle_USB2.0_14P, K1 G2RL-1A-E-HA DC5, K2 G2RL-1A-E-HA DC5, Q1 BTA16-600B, Q2 NMOS, Q3 NMOS, Q4 BTA16-600B, Q5 NMOS, Q6 NMOS, SW1 SW_Push, SW2 SW_Push, U1 ESP32-S3-WROOM-2, U2 AP7361C-33E, U3 LTV-354T, U4 FOD420, U5 74AHC1G08, U6 FOD420

Commit message: Almost done with schematic
Parts:
- added H1, H2: MountingHole_Pad_MP, symbol Mechanical:MountingHole_Pad_MP
- added J2: 54132-4062, 54132-4062_1, symbol 54132-4062:54132-4062
- added J3, J4, J6, J8: Conn_01x02_Pin, symbol Connector:Conn_01x02_Pin
- added J5, J7: Conn_01x03_Pin, symbol Connector:Conn_01x03_Pin
- added JP1, JP2: Jumper_2_Open, symbol Jumper:Jumper_2_Open
- added LED1: RGB, LED_SMD:LED_Cree-PLCC4_3.2x2.8mm_CCW, symbol LED:CLV1L-FKB
- added PS1: TMLM04105, Converter_ACDC:Converter_ACDC_TRACO_TMLM-04_THT, symbol Converter_ACDC:TMLM04105
- added Q7, Q8, Q9: NMOS, symbol Simulation_SPICE:NMOS
- added R19, R32: 10k, Resistor_SMD:R_0612_1632Metric_Pad1.18x3.40mm_HandSolder, symbol Device:R
- added R21, R22, R23, R24, R25, R26, R27, R31: R, Resistor_SMD:R_0612_1632Metric_Pad1.18x3.40mm_HandSolder, symbol Device:R
- added R28, R29, R30: 65, Resistor_SMD:R_0603_1608Metric_Pad0.98x0.95mm_HandSolder, symbol Device:R_Small
- added R33: 22k, Resistor_SMD:R_0612_1632Metric_Pad1.18x3.40mm_HandSolder, symbol Device:R
- added SW3: RotaryEncoder_Switch, symbol Device:RotaryEncoder_Switch
- added SW4: SW_SPDT, symbol Switch:SW_SPDT
- added TP10, TP11, TP12, TP13, TP14, TP15, TP16, TP17, TP18, TP19, TP2, TP20, TP21, TP22, TP23, TP24, TP25, TP26, TP27, TP3, TP4, TP5, TP6, TP7, TP8, TP9: TestPoint, symbol Connector:TestPoint
- added U7: INA122, symbol Amplifier_Instrumentation:INA128
- added U8: LM4041LP-ADJ, Package_TO_SOT_THT:TO-92_Inline, symbol Reference_Voltage:LM4041LP-ADJ
- added U9: LM358_DFN, Package_DFN_QFN:DFN-8-1EP_2x2mm_P0.5mm_EP1.05x1.75mm, symbol Amplifier_Operational:LM358_DFN
- R1, R10, R2, R3: footprint (none) -> Resistor_SMD:R_0603_1608Metric_Pad0.98x0.95mm_HandSolder
- R11, R12, R13, R14, R15, R18: footprint (none) -> Resistor_SMD:R_0612_1632Metric_Pad1.18x3.40mm_HandSolder
- TP1: footprint (none) -> Connector_PinHeader_2.54mm:PinHeader_1x01_P2.54mm_Horizontal
Connections:
- net IO17 is gone; now on net USR_HV_SWITCH: U1.10 (IO17)
- net IO18 is gone; now on net MCU_HV_CMD: U1.11 (IO18)
- net IO45 is gone; now on net BUZZER: U1.26 (IO45)
- net IO5 is gone; now on net AC_ZC: U1.5 (IO5)
- net IO6 is gone; now on net PUMP_TRIAC: U1.6 (IO6)
- net IO7 is gone; now on net BOILER_TRIAC: U1.7 (IO7)
- net IO8 is gone; now on net BUZZER: U1.12 (IO8)
- net +3.3V: now also J2.10, J2.12, J2.3, J2.33, LED1.1 (A), R19.2, R24.2, R31.2, SW4.1 (A), TP26.1, U7.7 (V+), U9.8 (V+)
- net +5V: now also J7.3 (Pin_3), TP27.1
- net 120VAC_HOT: now also PS1.5 (AC(L))
- net 120VAC_NEUTRAL: now also PS1.6 (AC(N))
- net 120VAC_NEUTRAL_SWITCHED: now also H2.MP, J5.1 (Pin_1)
- net AC_RELAYS: now also TP19.1
- net AC_ZC: now also TP23.1
- net BOILER_HOT_OUT: now also H1.MP
- net BOILER_TRIAC: now also TP25.1
- net GND: now also BZ1.2 (-), J2.1, J2.14, J2.15, J2.16, J2.17, J2.18, J2.19, J2.20, J2.21, J2.22, J2.23, J2.24, J2.25, J2.26, J2.27, J2.28, J2.29, J2.30, J2.34, J2.35, J2.36, J2.37, J2.40, J6.1 (Pin_1), J7.1 (Pin_1), PS1.3 (Vout-), Q7.3 (S), Q8.3 (S), Q9.3 (S), R22.2, R23.2, R26.1, R33.2, SW3.C, SW3.S2, SW4.3 (C), U7.4 (V-), U8.3 (A), U9.4 (V-), U9.5 (+), U9.9 (PAD)
- net IO0: now also TP13.1; no longer U1.27 (IO0)
- net IO21: now also J8.2 (Pin_2)
- net IO38: now also J8.1 (Pin_1)
- net PUMP_HOT_OUT: now also J5.3 (Pin_3)
- net PUMP_TRIAC: now also TP24.1
- net RST: now also TP14.1
- net RXD0/IO44: now also J4.1 (Pin_1)
- net TXD0/IO43: now also J4.2 (Pin_2)
- net USB_VBUS_Unprotected: now also JP1.1 (A); no longer F1.1
- net MCU_HV_CMD: now reaches U5.1
- net MCU_HV_CMD: now also TP20.1
- net USR_HV_SWITCH: now reaches U5.2
- net USR_HV_SWITCH: now also SW4.2 (B), TP15.1
- net BUZZER: now reaches BZ1.1 (+)
- net IO1 renamed LCD_CTP_INT
- net LCD_CTP_INT: now also J2.5, TP12.1
- net IO10 renamed DISPLAY_CS0
- net DISPLAY_CS0: now also J2.9, TP3.1
- net IO11 renamed DISPLAY_MOSI
- net DISPLAY_MOSI: now also J2.2, TP4.1
- net IO12 renamed DISPLAY_CLK
- net DISPLAY_CLK: now also J2.8, TP5.1
- net IO13 renamed DISPLAY_MISO
- net DISPLAY_MISO: now also J2.13, TP6.1
- net IO14 renamed DISPLAY_RESET
- net DISPLAY_RESET: now also J2.7, TP7.1
- net IO15 renamed DISPLAY_FRMARK
- net DISPLAY_FRMARK: now also J2.4, TP8.1
- net IO16 renamed PRESSURE_SIG_ANALOG
- net PRESSURE_SIG_ANALOG: now also R32.2, R33.1, TP22.1
- net IO2 renamed LCD_CTP_RST
- net LCD_CTP_RST: now also J2.31, TP11.1
- net IO3 renamed LCD_CTP_SCL
- net LCD_CTP_SCL: now also J2.6, TP10.1
- net IO4 renamed LCD_CTP_SDA
- net LCD_CTP_SDA: now also J2.32, TP9.1
- net IO46 renamed LED_R
- net LED_R: now also Q7.2 (G)
- net IO47 renamed LED_G
- net LED_G: now also Q8.2 (G)
- net IO48 renamed LED_B
- net LED_B: now also Q9.2 (G)
- net IO9 renamed DISPLAY_DC
- net DISPLAY_DC: now also J2.11, TP2.1
- new net: LED1.2 (RK), R28.1
- new net: Q7.1 (D), R28.2
- new net: F1.1, JP1.2 (B), JP2.2 (B)
- new net: R25.1, R26.2, U8.1 (FB)
- new net: Q9.1 (D), R30.2
- new net: R27.1, U7.1 (Rg)
- new net: R21.2, R22.1, U7.2 (-)
- new net: R27.2, U7.8 (Rg)
- new net: U9.6 (-), U9.7
- new net: LED1.3 (GK), R29.1
- new net: LED1.4 (BK), R30.1
- new net: R32.1, U9.1, U9.2 (-)
- new net: Q8.1 (D), R29.2
- new net ACDC_5V: JP2.1 (A), PS1.2 (Vout+)
- new net PRESSURE_SENSOR_IN: U9.3 (+)
- new net PRESSURE_SENSOR_SIG: J7.2 (Pin_2)
- new net ROTARYENC_A: SW3.A, TP17.1
- new net ROTARYENC_B: SW3.B, TP18.1
- new net ROTARYENC_SWITCH: R19.1, SW3.S1, TP16.1
- new net STEAM_VALVE_IN: J6.2 (Pin_2), R31.1
- new net THERMISTOR_IN: J3.2 (Pin_2), R21.1, R24.1, R25.2, U7.5 (Ref), U8.2 (K)
- new net THERMISTOR_OUT: J3.1 (Pin_1), R23.1, U7.3 (+)
- new net THERMISTOR_SIG_ANALOG: TP21.1, U1.27 (IO0), U7.6
- no-connect marks 0 -> 1
Other:
- note added: "AC-DC LV Power"
- note added: "Display SPI pins mapped to ESP32 FSPI Pins selected to bypass GPIO matrix"
- note added: "HV Connections"
- note added: "HV Control Switch"
- note added: "IOMUX for Fast SPI"
- note added: "Knob Encoder"
- note added: "LCD: 4DLCD-24320240-CTP-IPS"
- note added: "NTC Thermistor"
- note added: "OEM sensor connectors are B2B-XH?"
- note added: "Pressure Sensor Measurement"
- note added: "RGB LED"
- note added: "Relay Control"
- note added: "Sensor Connections"
- note added: "Set to use SPI mode via IM0 pin"
- note added: "Steam Valve Switch"
- note added: "TODO: Pressure Sensor"
- note added: "Thermistor Measurement"
- note added: "Unused IO"
- note added: "User Input"
- note added: "User Output (LCD)"
- note added: "Wheatstone Bridge + Instrumentation Amp"
- note removed: "Sensor connectors are B2B-XH?"
- moved on the sheet: BZ1, C1, C2, D1, D2, D4, D5, F1, K1, K2, Q1, Q2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

Commit message: Split into 2 board
Parts:
- J2: footprint 54132-4062_1 -> EspressoMachineHW:54132-4062_1
- R11, R12, R13, R14, R15, R18, R19, R21, R22, R23, R24, R25, R26, R27, R31, R32, R33: footprint Resistor_SMD:R_0612_1632Metric_Pad1.18x3.40mm_HandSolder -> Resistor_SMD:R_0603_1608Metric_Pad0.98x0.95mm_HandSolder
- TP1: footprint Connector_PinHeader_2.54mm:PinHeader_1x01_P2.54mm_Horizontal -> Connector_PinHeader_2.54mm:PinHeader_1x01_P2.54mm_Vertical
- TP10, TP11, TP12, TP13, TP14, TP15, TP16, TP17, TP18, TP19, TP2, TP20, TP21, TP22, TP23, TP24, TP25, TP26, TP27, TP3, TP4, TP5, TP6, TP7, TP8, TP9: footprint (none) -> Connector_PinHeader_2.54mm:PinHeader_1x01_P2.54mm_Vertical
Other:
- note added: "TODO: Wheatstone bridge and other resistor values Capacitor footprints Final measurements"
- note removed: "TODO: Pressure Sensor"
Changed lines of the file:
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@@
 	(text "HV AC"
 		(exclude_from_sim no)
-		(at 274.828 17.526 0)
+		(at 274.828 17.272 0)
 		(effects
 			(font
@@
 		)
 	)
-	(text "TODO: Pressure Sensor"
+	(text "TODO:\nWheatstone bridge and other resistor values\nCapacitor footprints\nFinal measurements"
 		(exclude_from_sim no)
 		(at 263.652 238.506 0)
@@
 			)
 		)
-		(property "Footprint" ""
+		(property "Footprint" "Connector_PinHeader_2.54mm:PinHeader_1x01_P2.54mm_Vertical"
 			(at 128.27 58.42 0)
 			(effects
@@
 			)
 		)
-		(property "Footprint" ""
+		(property "Footprint" "Connector_PinHeader_2.54mm:PinHeader_1x01_P2.54mm_Vertical"
 			(at 161.29 171.45 0)
 			(effects
@@
 			)
 		)
-		(property "Footprint" ""
+		(property "Footprint" "Connector_PinHeader_2.54mm:PinHeader_1x01_P2.54mm_Vertical"
 			(at 95.25 259.08 0)
 			(effects
@@
 			)
 		)
-		(property "Footprint" "Resistor_SMD:R_0612_1632Metric_Pad1.18x3.40mm_HandSolder"
+		(property "Footprint" "Resistor_SMD:R_0603_1608Metric_Pad0.98x0.95mm_HandSolder"
 			(at 130.302 218.44 90)
 			(effects
@@
 			)
 		)
-		(property "Footprint" "Resistor_SMD:R_0612_1632Metric_Pad1.18x3.40mm_HandSolder"
+		(property "Footprint" "Resistor_SMD:R_0603_1608Metric_Pad0.98x0.95mm_HandSolder"
 			(at 157.48 108.458 90)
 			(effects
@@
 			)
 		)
-		(property "Footprint" ""
+		(property "Footprint" "Connector_PinHeader_2.54mm:PinHeader_1x01_P2.54mm_Vertical"
 			(at 91.44 251.46 0)
 			(effects
@@
 			)
 		)
-		(property "Footprint" ""
+		(property "Footprint" "Connector_PinHeader_2.54mm:PinHeader_1x01_P2.54mm_Vertical"
 			(at 93.98 256.54 0)
 			(effects
@@
 			)
 		)
-		(property "Footprint" ""
+		(property "Footprint" "Connector_PinHeader_2.54mm:PinHeader_1x01_P2.54mm_Vertical"
 			(at 88.9 120.65 0)
 			(effects
@@
 			)
 		)
-		(property "Footprint" "Resistor_SMD:R_0612_1632Metric_Pad1.18x3.40mm_HandSolder"
+		(property "Footprint" "Resistor_SMD:R_0603_1608Metric_Pad0.98x0.95mm_HandSolder"
 			(at 384.048 162.56 90)
 			(effects
@@
 			)
 		)
-		(property "Footprint" ""
+		(property "Footprint" "Connector_PinHeader_2.54mm:PinHeader_1x01_P2.54mm_Vertical"
 			(at 35.56 219.71 0)
 			(effects
@@
 			)
 		)
-		(property "Footprint" "Resistor_SMD:R_0612_1632Metric_Pad1.18x3.40mm_HandSolder"
+		(property "Footprint" "Resistor_SMD:R_0603_1608Metric_Pad0.98x0.95mm_HandSolder"
 			(at 186.69 59.182 90)
 			(effects
@@
 			)
 		)
-		(property "Footprint" "Resistor_SMD:R_0612_1632Metric_Pad1.18x3.40mm_HandSolder"
+		(property "Footprint" "Resistor_SMD:R_0603_1608Metric_Pad0.98x0.95mm_HandSolder"
 			(at 141.478 250.19 90)
 			(effects
@@
 			)
 		)
-		(property "Footprint" ""
+		(property "Footprint" "Connector_PinHeader_2.54mm:PinHeader_1x01_P2.54mm_Vertical"
 			(at 34.29 217.17 0)
 			(effects
@@
 			)
 		)
-		(property "Footprint" ""
+		(property "Footprint" "Connector_PinHeader_2.54mm:PinHeader_1x01_P2.54mm_Vertical"
 			(at 405.13 177.8 0)
 			(effects
@@
 			)
 		)
-		(property "Footprint" ""
+		(property "Footprint" "Connector_PinHeader_2.54mm:PinHeader_1x01_P2.54mm_Vertical"
 			(at 135.89 97.79 0)
 			(effects
@@
 			)
 		)
-		(property "Footprint" ""
+		(property "Footprint" "Connector_PinHeader_2.54mm:PinHeader_1x01_P2.54mm_Vertical"
 			(at 90.17 248.92 0)
 			(effects
@@
 			)
 		)
-		(property "Footprint" ""
+		(property "Footprint" "Connector_PinHeader_2.54mm:PinHeader_1x01_P2.54mm_Vertical"
 			(at 85.09 151.13 0)
 			(effects
@@
 			)
 		)
-		(property "Footprint" ""
+		(property "Footprint" "Connector_PinHeader_2.54mm:PinHeader_1x01_P2.54mm_Vertical"
 			(at 88.9 246.38 0)
 			(effects
@@
 			)
 		)
-		(property "Footprint" ""
+		(property "Footprint" "Connector_PinHeader_2.54mm:PinHeader_1x01_P2.54mm_Vertical"
 			(at 140.97 137.16 0)
 			(effects
@@
 			)
 		)
-		(property "Footprint" ""
+		(property "Footprint" "Connector_PinHeader_2.54mm:PinHeader_1x01_P2.54mm_Vertical"
 			(at 135.89 161.29 0)
 			(effects
@@
 			)
 		)
-		(property "Footprint" ""
+		(property "Footprint" "Connector_PinHeader_2.54mm:PinHeader_1x01_P2.54mm_Vertical"
 			(at 218.44 191.77 0)
 			(effects
@@
 			)
 		)
-		(property "Footprint" "Resistor_SMD:R_0612_1632Metric_Pad1.18x3.40mm_HandSolder"
+		(property "Footprint" "Resistor_SMD:R_0603_1608Metric_Pad0.98x0.95mm_HandSolder"
 			(at 236.22 151.638 90)
 			(effects
@@
 			)
 		)
-		(property "Footprint" "Connector_PinHeader_2.54mm:PinHeader_1x01_P2.54mm_Horizontal"
+		(property "Footprint" "Connector_PinHeader_2.54mm:PinHeader_1x01_P2.54mm_Vertical"
 			(at 129.54 27.94 0)
 			(effects
@@
 			)
 		)
-		(property "Footprint" ""
+		(property "Footprint" "Connector_PinHeader_2.54mm:PinHeader_1x01_P2.54mm_Vertical"
 			(at 137.16 100.33 0)
 			(effects
@@
 			)
 		)
-		(property "Footprint" ""
+		(property "Footprint" "Connector_PinHeader_2.54mm:PinHeader_1x01_P2.54mm_Vertical"
 			(at 307.34 158.75 0)
 			(effects
@@
 			)
 		)
-		(property "Footprint" "Resistor_SMD:R_0612_1632Metric_Pad1.18x3.40mm_HandSolder"
+		(property "Footprint" "Resistor_SMD:R_0603_1608Metric_Pad0.98x0.95mm_HandSolder"
 			(at 143.002 218.44 90)
 			(effects
@@
 			)
 		)
-		(property "Footprint" "Resistor_SMD:R_0612_1632Metric_Pad1.18x3.40mm_HandSolder"
+		(property "Footprint" "Resistor_SMD:R_0603_1608Metric_Pad0.98x0.95mm_HandSolder"
 			(at 353.568 170.18 90)
 			(effects
@@
 			)
 		)
-		(property "Footprint" ""
+		(property "Footprint" "Connector_PinHeader_2.54mm:PinHeader_1x01_P2.54mm_Vertical"
 			(at 360.68 177.8 0)
 			(effects
@@
 			)
 		)
-		(property "Footprint" "Resistor_SMD:R_0612_1632Metric_Pad1.18x3.40mm_HandSolder"
+		(property "Footprint" "Resistor_SMD:R_0603_1608Metric_Pad0.98x0.95mm_HandSolder"
 			(at 234.95 102.108 90)
 			(effects
@@
 			)
 		)
-		(property "Footprint" ""
+		(property "Footprint" "Connector_PinHeader_2.54mm:PinHeader_1x01_P2.54mm_Vertical"
 			(at 36.83 222.25 0)
 			(effects
@@
 			)
 		)
-		(property "Footprint" "Resistor_SMD:R_0612_1632Metric_Pad1.18x3.40mm_HandSolder"
+		(property "Footprint" "Resistor_SMD:R_0603_1608Metric_Pad0.98x0.95mm_HandSolder"
 			(at 396.748 170.18 90)
 			(effects
@@
 			)
 		)
-		(property "Footprint" "Resistor_SMD:R_0612_1632Metric_Pad1.18x3.40mm_HandSolder"
+		(property "Footprint" "Resistor_SMD:R_0603_1608Metric_Pad0.98x0.95mm_HandSolder"
 			(at 340.868 162.56 90)
 			(effects
@@
 			)
 		)
-		(property "Footprint" ""
+		(property "Footprint" "Connector_PinHeader_2.54mm:PinHeader_1x01_P2.54mm_Vertical"
 			(at 38.1 224.79 0)
 			(effects
@@
 			)
 		)
-		(property "Footprint" "54132-4062_1"
+		(property "Footprint" "EspressoMachineHW:54132-4062_1"
 			(at 119.05 234.95 0)
 			(effects
@@
 			)
 		)
-		(property "Footprint" ""
+		(property "Footprint" "Connector_PinHeader_2.54mm:PinHeader_1x01_P2.54mm_Vertical"
 			(at 92.71 254 0)
 			(effects
@@
 			)
 		)
-		(property "Footprint" ""
+		(property "Footprint" "Connector_PinHeader_2.54mm:PinHeader_1x01_P2.54mm_Vertical"
 			(at 53.34 110.49 0)
 			(effects
@@
 			)
 		)
-		(property "Footprint" ""
+		(property "Footprint" "Connector_PinHeader_2.54mm:PinHeader_1x01_P2.54mm_Vertical"
 			(at 157.48 95.25 0)
 			(effects
@@
 			)
 		)
-		(property "Footprint" ""
+		(property "Footprint" "Connector_PinHeader_2.54mm:PinHeader_1x01_P2.54mm_Vertical"
 			(at 87.63 243.84 0)
 			(effects
@@
 			)
 		)
-		(property "Footprint" "Resistor_SMD:R_0612_1632Metric_Pad1.18x3.40mm_HandSolder"
+		(property "Footprint" "Resistor_SMD:R_0603_1608Metric_Pad0.98x0.95mm_HandSolder"
 			(at 207.772 185.42 90)
 			(effects
@@
 			)
 		)
-		(property "Footprint" "Resistor_SMD:R_0612_1632Metric_Pad1.18x3.40mm_HandSolder"
+		(property "Footprint" "Resistor_SMD:R_0603_1608Metric_Pad0.98x0.95mm_HandSolder"
 			(at 207.772 195.58 90)
 			(effects
@@
 			)
 		)
-		(property "Footprint" "Resistor_SMD:R_0612_1632Metric_Pad1.18x3.40mm_HandSolder"
+		(property "Footprint" "Resistor_SMD:R_0603_1608Metric_Pad0.98x0.95mm_HandSolder"
 			(at 141.478 266.7 90)
 			(effects
@@
 			)
 		)
-		(property "Footprint" "Resistor_SMD:R_0612_1632Metric_Pad1.18x3.40mm_HandSolder"
+		(property "Footprint" "Resistor_SMD:R_0603_1608Metric_Pad0.98x0.95mm_HandSolder"
 			(at 120.142 208.28 90)
 			(effects
@@
 			)
 		)
-		(property "Footprint" "Resistor_SMD:R_0612_1632Metric_Pad1.18x3.40mm_HandSolder"
+		(property "Footprint" "Resistor_SMD:R_0603_1608Metric_Pad0.98x0.95mm_HandSolder"
 			(at 141.478 259.08 90)
 			(effects
@@
 			)
 		)
-		(property "Footprint" "Resistor_SMD:R_0612_1632Metric_Pad1.18x3.40mm_HandSolder"
+		(property "Footprint" "Resistor_SMD:R_0603_1608Metric_Pad0.98x0.95mm_HandSolder"
 			(at 120.142 218.44 90)
 			(effects
@@
 			)
 		)
-		(property "Footprint" ""
+		(property "Footprint" "Connector_PinHeader_2.54mm:PinHeader_1x01_P2.54mm_Vertical"
 			(at 101.6 58.42 0)
 			(effects

Commit message: More work
Other:
- note added: "TODO: Wheatstone bridge and other resistor values Capacitor footprints Final measurements Thermistor 60hz LPF"
- note removed: "TODO: Wheatstone bridge and other resistor values Capacitor footprints Final measurements"
Changed lines of the file:
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@@
 		)
 	)
-	(text "TODO:\nWheatstone bridge and other resistor values\nCapacitor footprints\nFinal measurements"
+	(text "TODO:\nWheatstone bridge and other resistor values\nCapacitor footprints\nFinal measurements\nThermistor 60hz LPF"
 		(exclude_from_sim no)
-		(at 263.652 238.506 0)
+		(at 262.89 248.666 0)
 		(effects
 			(font

Commit message: Boards finalized and ordered
Parts:
- removed C1, C2: 0.01u, symbol Device:C_Polarized
- removed D4, D5: D_Zener, symbol Device:D_Zener
- removed H1, H2: MountingHole_Pad_MP, symbol Mechanical:MountingHole_Pad_MP
- removed J2: 54132-4062, EspressoMachineHW:54132-4062_1, symbol 54132-4062:54132-4062
- removed J5, J7: Conn_01x03_Pin, symbol Connector:Conn_01x03_Pin
- removed J6, J8: Conn_01x02_Pin, symbol Connector:Conn_01x02_Pin
- removed K1, K2: G2RL-1A-E-HA DC5, Relay_THT:Relay_SPST_Omron_G2RL-1A-E, symbol Relay:G2RL-1A-E
- removed PS1: TMLM04105, Converter_ACDC:Converter_ACDC_TRACO_TMLM-04_THT, symbol Converter_ACDC:TMLM04105
- removed Q1, Q4: BTA16-600B, Package_TO_SOT_THT:TO-220-3_Vertical, symbol Triac_Thyristor:BTA16-600B
- removed Q3, Q5, Q6: NMOS, symbol Simulation_SPICE:NMOS
- removed R10, R14, R18: 10k, Resistor_SMD:R_0603_1608Metric_Pad0.98x0.95mm_HandSolder, symbol Device:R
- removed R11, R15: 65, Resistor_SMD:R_0603_1608Metric_Pad0.98x0.95mm_HandSolder, symbol Device:R
- removed R12, R13: 1k, Resistor_SMD:R_0603_1608Metric_Pad0.98x0.95mm_HandSolder, symbol Device:R
- removed R16: 360, symbol Device:R
- removed R17: 330, symbol Device:R
- removed R20, R7: 39, symbol Device:R
- removed R21, R22, R25, R26, R27: R, Resistor_SMD:R_0603_1608Metric_Pad0.98x0.95mm_HandSolder, symbol Device:R
- removed R8, R9: 47k, symbol Device:R
- removed TP10, TP11, TP12, TP13, TP14, TP16, TP20, TP21, TP23, TP24, TP25, TP4, TP5, TP6, TP7, TP9: TestPoint, Connector_PinHeader_2.54mm:PinHeader_1x01_P2.54mm_Vertical, symbol Connector:TestPoint
- removed U3: LTV-354T, Package_SO:SO-4_4.4x3.6mm_P2.54mm, symbol Isolator:LTV-354T
- removed U4, U6: FOD420, Package_DIP:DIP-6_W7.62mm, symbol Relay_SolidState:FOD420
- removed U7: INA122, symbol Amplifier_Instrumentation:INA128
- removed U8: LM4041LP-ADJ, Package_TO_SOT_THT:TO-92_Inline, symbol Reference_Voltage:LM4041LP-ADJ
- added C1: 100n, Capacitor_SMD:C_0603_1608Metric_Pad1.08x0.95mm_HandSolder, symbol Device:C
- added C2: 47n, Capacitor_SMD:C_0603_1608Metric_Pad1.08x0.95mm_HandSolder, symbol Device:C
- added H1, H2, H3, H4: MountingHole_Pad, MountingHole:MountingHole_3.2mm_M3_DIN965, symbol Mechanical:MountingHole_Pad
- added H5, H6, H7, H8: MountingHole_Pad, MountingHole:MountingHole_3.2mm_M3_DIN965_Pad, symbol Mechanical:MountingHole_Pad
- added J2: Conn_01x04_Pin, Connector_PinSocket_2.54mm:PinSocket_1x04_P2.54mm_Vertical, symbol Connector:Conn_01x04_Pin
- added J5: Conn_01x08_Pin, Connector_JST:JST_PH_B8B-PH-K_1x08_P2.00mm_Vertical, symbol Connector:Conn_01x08_Pin
- added J6, J7: Conn_01x14_Pin, Connector_PinSocket_2.54mm:PinSocket_1x14_P2.54mm_Vertical, symbol Connector:Conn_01x14_Pin
- added JP3, JP4: Jumper_2_Open, Jumper:SolderJumper-2_P1.3mm_Open_Pad1.0x1.5mm, symbol Jumper:Jumper_2_Open
- added Q1: NMOS, Package_TO_SOT_SMD:SOT-23, symbol Simulation_SPICE:NMOS
- added U3: LM358_DFN, Package_SO:SOIC-8_3.9x4.9mm_P1.27mm, symbol Amplifier_Operational:LM358_DFN
- added U6: LM4040A25IDCKR, Package_TO_SOT_SMD:SOT-353_SC-70-5, symbol Reference_Voltage:LM4040DCK-2.5
- BZ1: footprint (none) -> Buzzer_Beeper:Buzzer_TDK_PS1240P02BT_D12.2mm_H6.5mm
- F1: footprint (none) -> Fuse:Fuse_0603_1608Metric_Pad1.05x0.95mm_HandSolder
- J1: footprint (none) -> Connector_USB:USB_C_Receptacle_GCT_USB4110
- J3: footprint (none) -> Connector_JST:JST_XH_B2B-XH-AM_1x02_P2.50mm_Vertical
- J4: footprint (none) -> Connector_PinSocket_2.54mm:PinSocket_1x02_P2.54mm_Vertical
- JP1, JP2: footprint (none) -> Jumper:SolderJumper-2_P1.3mm_Open_Pad1.0x1.5mm
- Q2, Q7, Q8, Q9: footprint (none) -> Package_TO_SOT_SMD:SOT-23
- R23, R31: value R -> 10k
- R24: value R -> 3k
- R28, R29, R30, R4: value 65 -> 65R
- R5: value 360 -> 47k; footprint (none) -> Resistor_SMD:R_0603_1608Metric_Pad0.98x0.95mm_HandSolder
- R6: value 330 -> 47k; footprint (none) -> Resistor_SMD:R_0603_1608Metric_Pad0.98x0.95mm_HandSolder
- SW1, SW2: footprint (none) -> Button_Switch_SMD:SW_Push_1P1T_NO_6x6mm_H9.5mm
- SW3: value RotaryEncoder_Switch -> PEC11R-4215K-S0012; footprint (none) -> Rotary_Encoder:RotaryEncoder_Alps_EC11E-Switch_Vertical_H20mm
- SW4: footprint (none) -> Button_Switch_THT:SW_Slide_SPDT_Straight_CK_OS102011MS2Q
- U5: value 74AHC1G08 -> 74AHC1G08GW,125; footprint (none) -> Package_TO_SOT_SMD:SOT-353_SC-70-5_Handsoldering
- U9: footprint Package_DFN_QFN:DFN-8-1EP_2x2mm_P0.5mm_EP1.05x1.75mm -> Package_SO:SOIC-8_3.9x4.9mm_P1.27mm
Connections:
- net 120VAC_HOT_SWITCHED is gone; now on an unnamed net: R5.2
- net IO0 is gone; now on net BUZZER: SW1.1
- net IO38 is gone; now on net LCD_CTP_SDA: U1.31 (IO38)
- net +3.3V: now also U3.8 (V+)
- net +5V: now also J6.14 (Pin_14), J7.14 (Pin_14)
- net ACDC_5V: now also J5.1 (Pin_1)
- net AC_RELAYS: now also J5.6 (Pin_6)
- net AC_ZC: now also J5.3 (Pin_3)
- net BOILER_TRIAC: now also J5.7 (Pin_7)
- net BUZZER: now also Q2.2 (G), U1.27 (IO0); no longer BZ1.1 (+), U1.12 (IO8), U1.26 (IO45)
- net DISPLAY_CLK: now also J6.8 (Pin_8), J7.8 (Pin_8)
- net DISPLAY_CS0: now also J6.12 (Pin_12), J7.12 (Pin_12); no longer TP3.1
- net DISPLAY_DC: now also J6.10 (Pin_10), J7.10 (Pin_10); no longer TP2.1
- net DISPLAY_MISO: now also J6.6 (Pin_6), J7.6 (Pin_6)
- net DISPLAY_MOSI: now also J6.9 (Pin_9), J7.9 (Pin_9)
- net DISPLAY_RESET: now also J6.11 (Pin_11), J7.11 (Pin_11)
- net GND: now also TP2.1, TP3.1, C2.2, H1.1, H2.1, H3.1, H4.1, H5.1, H6.1, H7.1, H8.1, J5.8 (Pin_8), J6.13 (Pin_13), J7.13 (Pin_13), Q1.3 (S), U3.4 (V-), U3.9 (PAD), U6.1 (A)
- net LCD_CTP_INT: now also J6.2 (Pin_2), J7.2 (Pin_2)
- net LCD_CTP_RST: now also U1.4 (IO4), J6.4 (Pin_4), J7.4 (Pin_4); no longer U1.38 (IO2)
- net LCD_CTP_SCL: now also J6.5 (Pin_5), J7.5 (Pin_5)
- net LCD_CTP_SDA: now also J6.3 (Pin_3), J7.3 (Pin_3); no longer U1.4 (IO4)
- net MCU_HV_CMD: now also U5.2; no longer U5.1
- net MTCK/IO39: now also J2.4 (Pin_4)
- net MTDI/IO41: now also J2.2 (Pin_2)
- net MTDO/IO40: now also J2.3 (Pin_3)
- net MTMS/IO42: now also J2.1 (Pin_1)
- net PRESSURE_SENSOR_IN: now also J5.2 (Pin_2)
- net PUMP_TRIAC: now also J5.4 (Pin_4)
- net ROTARYENC_A: now also JP3.1 (A)
- net ROTARYENC_B: now also JP4.2 (B)
- net ROTARYENC_SWITCH: now also U1.10 (IO17)
- net RXD0/IO44: now also JP4.1 (A)
- net THERMISTOR_IN: now also U6.3 (K)
- net THERMISTOR_OUT: now also U3.3 (+)
- net THERMISTOR_SIG_ANALOG: now also TP8.1, U1.38 (IO2), C1.1, U3.6 (-), U3.7; no longer U1.27 (IO0)
- net TXD0/IO43: now also JP3.2 (B)
- net USR_HV_SWITCH: now also U1.8 (IO15), U5.1; no longer U1.10 (IO17), U5.2
- net at R6.1: now also C1.2
- net at Q2.1 (D): now also BZ1.1 (+)
- net at R5.1: now also U3.1, U3.2 (-)
- removed net DISPLAY_FRMARK: TP8.1, U1.8 (IO15)
- net IO21 renamed ~{LCD_LED}
- net ~{LCD_LED}: now also Q1.2 (G)
- net PUMP_HOT_OUT: no longer names the net of R6.2
- net PUMP_HOT_OUT: now also C2.1, U3.5 (+)
- net STEAM_VALVE_IN renamed STEAM_VALVE_SIG
- net STEAM_VALVE_SIG: now also U1.26 (IO45), J5.5 (Pin_5)
- new net: J6.7 (Pin_7), J7.7 (Pin_7), Q1.1 (D)
- new net SD_CS: J6.1 (Pin_1), J7.1 (Pin_1), U1.12 (IO8)
- no-connect marks 1 -> 0
Other:
- note added: "100k NTC Thermistor"
- note added: "60hz Active LPF (Actually ~48Hz)"
- note added: "Board Mounting holes"
- note added: "Debug header Don't populate unless needed"
- note added: "ESP32 ADC: 12-bit SAR ~150mV - 2450mV Range (12dB attenuation)"
- note added: "LCD Mounting holes"
- note added: "New screen:"
- note added: "Op-Amps: LM358LVIDR"
- note added: "PS1240P02BT"
- note added: "Push buttons: 2-1977223-9"
- note added: "SLW-12689-4A-N-D (short) or SLW-121456-3A-N-D (long)"
- note added: "Steam Valve Switch Pullup"
- note added: "TODO: Final measurements Inter-board connections"
- note added: "Voltage divider + Buffer"
- note added: "https://www.amazon.com/Hosyond-320x480-Capacitive-Display-Mega2560/dp/B0CRGQN58D?pd_rd_w=MfTtT&content-id=amzn1.sym.cd152278-debd-42b9-91b9-6f271389fda7&pf_rd_p=cd152278-debd-42b9-91b9-6f271389fda7&pf_rd_r=4CVHM0RG5QGXJTRP6XDY&pd_rd_wg=Nnetp&pd_rd_r=2bbf2a5e-2d15-4c26-bcf4-4226e2b3f481&pd_rd_i=B0CRGQN58D&th=1"
- note removed: "AC-DC LV Power"
- note removed: "Boiler Control"
- note removed: "Boiler is soldered"
- note removed: "HV AC"
- note removed: "HV Connections"
- note removed: "LCD: 4DLCD-24320240-CTP-IPS"
- note removed: "LV DC"
- note removed: "Main HV Control"
- note removed: "Pump Control"
- note removed: "Pump connector is B3P-VH?"
- note removed: "Set to use SPI mode via IM0 pin"
- note removed: "Steam Valve Switch"
- note removed: "Switch both in case of reverse polarity (ex. reversed plug)"
- note removed: "TODO: Wheatstone bridge and other resistor values Capacitor footprints Final measurements Thermistor 60hz LPF"
- note removed: "Triac Control"
- note removed: "Unused IO"
- note removed: "Wheatstone Bridge + Instrumentation Amp"
- note removed: "Zero-Crossing Detection"
- moved on the sheet: BZ1, J3, J4, LED1, Q7, Q8, Q9, R19, R28, R29, R30, R31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

Commit message: Added issues
Other:
- note added: "Things that are wrong: SOT-23 MOSFET footprint has gate and source swapped -> they burn out when driven Switch schematic is different from part"
