File: HVBoard/HVBoard.kicad_pcb (KiCad board)
At the start: 2 copper layers, 100 x 60 mm, 19 parts, among them J2 Conn_01x08_Pin, K1 G2RL-1A-E-HA DC5, K2 G2RL-1A-E-HA DC5, Q3 BTA16-600B, Q5 BTA16-600B, U1 LTV-354T, U2 FOD420, U3 FOD420

Commit message: More work
Parts:
- removed PS1: TMLM04105, Converter_ACDC:Converter_ACDC_TRACO_TMLM-04_THT
- added C1: 0.01u, Capacitor_THT:C_Rect_L13.0mm_W4.0mm_P10.00mm_FKS3_FKP3_MKS4, F.Cu at (-25.5, 15.4)
- added C3: 0.01u, Capacitor_THT:C_Rect_L13.0mm_W4.0mm_P10.00mm_FKS3_FKP3_MKS4, F.Cu at (-25.5, 21.0)
- added H5: MountingHole, MountingHole:MountingHole_3.2mm_M3, F.Cu at (23.0, 47.0)
- added H6: MountingHole, MountingHole:MountingHole_3.2mm_M3, F.Cu at (91.0, 47.0)
- added J1: Conn_01x08_Pin, Connector_PinHeader_2.54mm:PinHeader_1x08_P2.54mm_Vertical, F.Cu at (-17.5, 42.7)
- added J3: B3P-VH__LF__SN_, HWBoard:HDRV3W114P0X396_1X3_1182X850X1090P, F.Cu at (54.6, 17.0)
- added Q1: NMOS, Package_TO_SOT_SMD:SOT-23, F.Cu at (72.2, 61.2)
- added Q2: NMOS, Package_TO_SOT_SMD:SOT-23, F.Cu at (56.9, 61.5)
- added Q4: NMOS, Package_TO_SOT_SMD:SOT-23, F.Cu at (105.0, 60.1)
- added Q6: NMOS, Package_TO_SOT_SMD:SOT-23, F.Cu at (91.0, 61.0)
- added R11: 360, Resistor_SMD:R_1206_3216Metric_Pad1.30x1.75mm_HandSolder, F.Cu at (17.6, -23.6)
- added R13: 39, Resistor_THT:R_Axial_DIN0207_L6.3mm_D2.5mm_P10.16mm_Horizontal, F.Cu at (134.3, 35.0)
- added R14: 330, Resistor_SMD:R_1206_3216Metric_Pad1.30x1.75mm_HandSolder, F.Cu at (17.6, -20.3)
- added R16: R, Resistor_SMD:R_0603_1608Metric_Pad0.98x0.95mm_HandSolder, F.Cu at (-13.0, 41.6)
- added R3: 47k, Resistor_SMD:R_1206_3216Metric_Pad1.30x1.75mm_HandSolder, F.Cu at (17.6, -36.8)
- added R5: 47k, Resistor_SMD:R_1206_3216Metric_Pad1.30x1.75mm_HandSolder, F.Cu at (17.6, -33.5)
- added R6: 360, Resistor_SMD:R_1206_3216Metric_Pad1.30x1.75mm_HandSolder, F.Cu at (17.6, -30.2)
- added R8: 39, Resistor_THT:R_Axial_DIN0207_L6.3mm_D2.5mm_P10.16mm_Horizontal, F.Cu at (134.3, 30.9)
- added R9: 330, Resistor_SMD:R_1206_3216Metric_Pad1.30x1.75mm_HandSolder, F.Cu at (17.6, -26.9)
- added U4: 5V700mA 3.5W, wx-dc12003:WX-DC12003, B.Cu at (39.0, 36.0)
- moved R10 135.9 mm to (102.4, 64.5), turned to 90 degrees
- moved R15 121.0 mm to (88.0, 64.4), turned to 90 degrees
- moved R1 116.8 mm to (69.7, 65.3), turned to 90 degrees
- moved R2 104.0 mm to (53.4, 65.5), turned to 90 degrees
- moved J2 54.5 mm to (37.5, 68.0), turned to -90 degrees
- moved Q5 50.6 mm to (82.4, 15.5), turned to 0 degrees
- moved Q3 48.2 mm to (71.4, 15.5), turned to 0 degrees
- moved U1 23.9 mm to (70.5, 37.1), turned to -90 degrees
- moved U2 23.1 mm to (96.4, 45.0), turned to 90 degrees
- moved K1 18.8 mm to (84.0, 54.0), turned to 180 degrees
- moved K2 17.5 mm to (62.2, 54.0), turned to 180 degrees
- moved U3 16.1 mm to (105.0, 45.0), turned to 90 degrees
Connections:
- K1 pad 13: /120VAC_HOT_SWITCHED -> 120VAC_HOT
- K1 pad 14: 120VAC_HOT -> /120VAC_HOT_SWITCHED
- K2 pad 13: /120VAC_NEUTRAL_SWITCHED -> 120VAC_NEUTRAL
- K2 pad 14: 120VAC_NEUTRAL -> /120VAC_NEUTRAL_SWITCHED
Routing:
- net /120VAC_HOT_SWITCHED: track 0.00 -> 36.3 mm
- net /PUMP_HOT_OUT: track 0.00 -> 26.7 mm
- net Net-(D2-A): track 0.00 -> 6.64 mm
- net Net-(D1-A): track 0.00 -> 6.64 mm
- net Net-(Q4-G): track 0.00 -> 5.13 mm
- net Net-(Q6-G): track 0.00 -> 4.29 mm
- net Net-(Q2-G): track 0.00 -> 4.06 mm
- net Net-(Q6-D): track 0.00 -> 3.71 mm
- net Net-(Q4-D): track 0.00 -> 3.67 mm
- net Net-(Q1-G): track 0.00 -> 2.90 mm
Other:
- board size 100 x 60 mm -> 117 x 60 mm
- board text added: "120VAC HV"
- board text added: "5VDC LV"
- board text added: "Boiler"
- board text added: "L"
- board text added: "N"
- board text added: "UP"

Commit message: More HV work
Parts:
- removed K2: G2RL-1A-E-HA DC5, Relay_THT:Relay_SPST_Omron_G2RL-1A-E
- removed Q2: NMOS, Package_TO_SOT_SMD:SOT-23
- added D1: D_Zener, Diode_SMD:D_SOD-123, F.Cu at (131.8, 46.0)
- added D2: PTVS6V0S1UR-QX, Diode_SMD:Nexperia_CFP3_SOD-123W, F.Cu at (103.0, 63.6)
- added D3: MP01EA06, Diode_SMD:D_SOD-123, F.Cu at (103.1, 60.3)
- added D4: LED, LED_SMD:LED_0603_1608Metric, F.Cu at (102.2, 66.5)
- added J4: Conn_01x02_Pin, Connector_JST:JST_XH_B2B-XH-AM_1x02_P2.50mm_Vertical, F.Cu at (18.0, 60.5)
- added J5: Conn_01x02_Pin, Connector_JST:JST_XH_B2B-XH-AM_1x02_P2.50mm_Vertical, F.Cu at (29.0, 63.5)
- added J6: Conn_01x03_Pin, Connector_JST:JST_XH_B3B-XH-AM_1x03_P2.50mm_Vertical, F.Cu at (35.5, 81.0)
- added J7: Screw_Terminal_01x02, TerminalBlock:TerminalBlock_bornier-2_P5.08mm, F.Cu at (62.4, 38.0)
- added J8: Screw_Terminal_01x02, TerminalBlock:TerminalBlock_bornier-2_P5.08mm, F.Cu at (106.5, 17.0)
- added R17: 20k, Resistor_SMD:R_0603_1608Metric_Pad0.98x0.95mm_HandSolder, F.Cu at (97.7, 67.0)
- added TP6: TestPoint, Connector_PinHeader_2.54mm:PinHeader_1x01_P2.54mm_Vertical, F.Cu at (97.8, 60.9)
- J1, J2: footprint Connector_PinHeader_2.54mm:PinHeader_1x08_P2.54mm_Vertical -> Connector_JST:JST_PH_B8B-PH-K_1x08_P2.00mm_Vertical
- R12, R7: value 65 -> 220
- R14, R9: moved to B.Cu
- R2: value 10k -> 220; footprint Resistor_SMD:R_0603_1608Metric_Pad0.98x0.95mm_HandSolder -> Resistor_SMD:R_0603_1608Metric
- U4: moved to F.Cu
- moved C1 123.8 mm to (98.0, 24.0)
- moved R11 103.8 mm to (100.0, 39.5), turned to 180 degrees
- moved R14 100.2 mm to (103.0, 32.0), turned to 90 degrees
- moved J2 90.5 mm to (128.0, 69.5)
- moved C3 88.1 mm to (62.5, 18.0), turned to -90 degrees
- moved R3 81.9 mm to (51.0, 38.0), turned to 90 degrees
- moved R6 76.7 mm to (55.5, 36.5), turned to 90 degrees
- moved R5 75.2 mm to (47.5, 35.5), turned to 90 degrees
- moved R9 73.7 mm to (74.0, 20.5), turned to 180 degrees
- moved R8 67.4 mm to (67.0, 32.6), turned to 90 degrees
- moved R2 44.2 mm to (97.5, 64.5), turned to 0 degrees
- moved U2 43.9 mm to (52.9, 50.8)
- moved R13 39.9 mm to (94.5, 32.2), turned to 90 degrees
- moved Q1 39.1 mm to (60.8, 98.7)
- moved R15 39.1 mm to (76.6, 101.8)
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Connections:
- J1 pad 1: unconnected-(J1-Pin_1-Pad1) -> /THERMISTOR_IN
- J1 pad 2: unconnected-(J1-Pin_2-Pad2) -> /THERMISTOR_OUT
- J2 pad 2: +3.3V -> /AC_RELAYS
- J2 pad 3: /ACDC_5V -> /AC_ZC
- J2 pad 4: /AC_RELAYS -> /PUMP_TRIAC
- J2 pad 5: /AC_ZC -> /BOILER_TRIAC
- J2 pad 6: /PUMP_TRIAC -> /STEAM_VALVE_IN
- J2 pad 7: /BOILER_TRIAC -> /PRESSURE_SENSOR_SIG
- J3 pad 3: /120VAC_NEUTRAL_SWITCHED -> 120VAC_NEUTRAL
- R12 pad 1: +3.3V -> +5V
- R2 pad 1: /AC_RELAYS -> +5V
- R4 pad 1: +3.3V -> /AC_ZC
- R4 pad 2: /AC_ZC -> +5V
- R5 pad 2: /120VAC_NEUTRAL_SWITCHED -> 120VAC_NEUTRAL
- R7 pad 1: +3.3V -> +5V
Routing:
- net Net-(Q3-G): track 0.00 -> 60.9 mm
- net 120VAC_HOT: track 0.00 -> 24.5 mm
- net 120VAC_NEUTRAL: track 0.00 -> 20.1 mm, vias 0 -> 1
- net /PUMP_HOT_OUT: track 26.7 -> 7.91 mm
- net Net-(Q5-G): track 0.00 -> 13.7 mm
- net /120VAC_HOT_SWITCHED: track 36.3 -> 27.1 mm
- net Net-(R5-Pad1): track 0.00 -> 6.97 mm
- net Net-(D2-A): track 6.64 -> 0.00 mm
- net Net-(R6-Pad1): track 0.00 -> 6.55 mm
- net /BOILER_HOT_OUT: track 0.00 -> 5.47 mm
- net Net-(R3-Pad1): track 0.00 -> 4.86 mm
- net Net-(R11-Pad1): track 0.00 -> 4.08 mm
- net Net-(D4-A): track 4.06 -> 0.00 mm
Other:
- board size 117 x 60 mm -> 128.5 x 77.5 mm
- board text added: "<- High current path ->"
- board text added: "Pump"
- board text removed: "Boiler"

Commit message: More HV work
Parts:
- removed J1: Conn_01x08_Pin, Connector_JST:JST_PH_B8B-PH-K_1x08_P2.00mm_Vertical
- removed R16: R, Resistor_SMD:R_0603_1608Metric_Pad0.98x0.95mm_HandSolder
- added F1: 1A, Fuse:Fuse_0603_1608Metric_Pad1.05x0.95mm_HandSolder, F.Cu at (46.6, 62.0)
- added J9: Conn_01x02_Pin, Connector_JST:JST_XH_B2B-XH-AM_1x02_P2.50mm_Vertical, F.Cu at (-7.90, 31.0)
- added JP1: Jumper_2_Open, Jumper:SolderJumper-2_P1.3mm_Open_Pad1.0x1.5mm, F.Cu at (45.0, 59.5)
- added R18: 10k, Resistor_SMD:R_0603_1608Metric_Pad0.98x0.95mm_HandSolder, F.Cu at (62.5, 63.0)
- added R19: 20k, Resistor_SMD:R_0603_1608Metric_Pad0.98x0.95mm_HandSolder, F.Cu at (63.5, 59.1)
- moved R12 125.2 mm to (99.0, 51.0)
- moved BOILER 121.6 mm to (93.0, 60.0)
- moved TP2 116.4 mm to (65.5, 78.5)
- moved AC_ZC 103.3 mm to (57.5, 63.5)
- moved R4 93.4 mm to (50.0, 56.9), turned to -90 degrees
- moved R7 91.6 mm to (53.0, 53.9), turned to 90 degrees
- moved J2 74.0 mm to (54.0, 67.5), turned to 0 degrees
- moved D2 57.6 mm to (45.5, 66.5), turned to -90 degrees
- moved Q4 55.7 mm to (57.5, 55.0), turned to 0 degrees
- moved D1 54.9 mm to (79.5, 62.5), turned to 180 degrees
- moved R10 54.5 mm to (58.0, 58.5)
- moved D3 51.6 mm to (51.5, 62.0), turned to 180 degrees
- moved R15 51.0 mm to (101.5, 57.4)
- moved R17 50.6 mm to (49.1, 53.0), turned to 180 degrees
- moved Q6 50.5 mm to (104.5, 54.6)
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- renumbered TP1 to AC_ZC, TP3 to BOILER
Routing:
- net /STEAM_VALVE_IN: track 0.00 -> 46.5 mm, vias 0 -> 1
- net /BOILER_TRIAC: track 0.00 -> 45.2 mm, vias 0 -> 1
- net /PRESSURE_SENSOR_SIG: track 0.00 -> 30.2 mm
- net /AC_ZC: track 0.00 -> 20.5 mm
- net /AC_RELAYS: track 0.00 -> 17.7 mm
- net /ACDC_5V: track 0.00 -> 10.8 mm
- net /PUMP_TRIAC: track 0.00 -> 8.92 mm
- net Net-(D2-K): track 0.00 -> 6.54 mm
- net +5V: track 0.00 -> 5.14 mm
- net Net-(R12-Pad2): track 0.00 -> 3.20 mm
- net Net-(D1-A): track 6.64 -> 9.54 mm
- net Net-(Q4-G): track 5.13 -> 2.23 mm
- net Net-(JP1-B): track 0.00 -> 2.54 mm
- net Net-(R7-Pad2): track 0.00 -> 2.23 mm
- net GND: track 0.00 -> 0.95 mm
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
Commit message: More HV work
Parts:
- added R16: 10k, Resistor_SMD:R_0603_1608Metric_Pad0.98x0.95mm_HandSolder, F.Cu at (75.1, 66.5)
- added R20: 10k, Resistor_SMD:R_0603_1608Metric_Pad0.98x0.95mm_HandSolder, F.Cu at (54.1, 58.0)
- added R21: 10k, Resistor_SMD:R_0603_1608Metric_Pad0.98x0.95mm_HandSolder, F.Cu at (104.5, 57.5)
- R1: value 10k -> 1k
- R14, R9: moved to F.Cu
- moved J9 45.0 mm to (21.0, 65.5), turned to -90 degrees
- moved TP6 40.5 mm to (49.0, 66.5)
- moved TP2 20.3 mm to (62.0, 58.5)
- moved R2 18.7 mm to (79.2, 68.0)
- moved D4 17.8 mm to (84.5, 68.0), turned to 180 degrees
- moved TP3 6.10 mm to (96.5, 65.0)
- moved R14 5.39 mm to (105.0, 37.0), turned to -90 degrees
- moved R19 4.98 mm to (66.6, 63.0), turned to 0 degrees
- moved J4 3.61 mm to (20.0, 57.5), turned to 0 degrees
- moved C3 2.50 mm to (62.5, 20.5)
- moved R5 1.95 mm to (47.5, 37.5)
- moved J5 1.50 mm to (30.5, 63.5)
- moved R11 1.50 mm to (100.0, 38.0)
- moved TP1 0.71 mm to (57.0, 63.0)
- moved R13 0.34 mm to (94.5, 32.5)
- renumbered AC_ZC to TP1, BOILER to TP3
Connections:
- net /ACDC_5V renamed Net-(JP1-A)
- net /THERMISTOR_IN renamed Net-(J4-Pin_2)
- net /THERMISTOR_OUT renamed Net-(J4-Pin_1)
- TP6 pad 1: Net-(D2-K) -> +5V
Routing:
- net GND: track 0.95 -> 124.6 mm, vias 0 -> 3
- net +5V: track 5.14 -> 95.7 mm, vias 0 -> 3
- net Net-(Q3-G): track 60.9 -> 90.8 mm, vias 0 -> 1
- net Net-(J4-Pin_1): track 0.00 -> 17.6 mm
- net /BOILER_HOT_OUT: track 5.47 -> 15.8 mm
- net Net-(J4-Pin_2): track 0.00 -> 8.62 mm
- net /PRESSURE_SENSOR_SIG: track 30.2 -> 37.1 mm
- net /PUMP_TRIAC: track 8.92 -> 14.2 mm
- net Net-(D4-A): track 0.00 -> 3.71 mm
- net Net-(Q4-G): track 2.23 -> 4.73 mm
- net Net-(Q6-G): track 3.66 -> 6.14 mm
- net Net-(Q5-G): track 13.7 -> 11.3 mm
- net Net-(R5-Pad1): track 6.97 -> 4.96 mm
- net Net-(Q1-G): track 3.24 -> 5.20 mm
- net Net-(R11-Pad1): track 4.08 -> 5.58 mm
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- added copper zone on B.Cu, net /120VAC_HOT_SWITCHED
- added copper zone on F.Cu, net /120VAC_HOT_SWITCHED
- added copper zone on B.Cu, net /BOILER_HOT_OUT
- added copper zone on F.Cu, net /BOILER_HOT_OUT
- added copper zone on F.Cu, net /PUMP_HOT_OUT
- added copper zone on F.Cu, net 120VAC_HOT
- added copper zone on B.Cu, net 120VAC_NEUTRAL
- added copper zone on B.Cu, net Net-(C1-Pad1)
- added copper zone on F.Cu, net Net-(C1-Pad1)
- added copper zone on F.Cu, net Net-(C3-Pad1)
Other:
- board size 128.5 x 77.5 mm -> 106 x 77.5 mm
- board text added: "Boiler"
- board text added: "Mains In"
- board text removed: "<- High current path ->"
- board text removed: "LV 5VDC"

Commit message: Reddit feedback integrated into HV board
Parts:
- ACDC Converter: renamed from U4
- C1, C3: footprint Capacitor_THT:C_Rect_L13.0mm_W4.0mm_P10.00mm_FKS3_FKP3_MKS4 -> Capacitor_THT:C_Disc_D11.0mm_W5.0mm_P7.50mm
Connections:
- J2 pad 2: /AC_RELAYS -> /PRESSURE_SENSOR_SIG
- J2 pad 5: /BOILER_TRIAC -> /STEAM_VALVE_IN
- J2 pad 6: /STEAM_VALVE_IN -> /AC_RELAYS
- J2 pad 7: /PRESSURE_SENSOR_SIG -> /BOILER_TRIAC
Routing:
- net /PRESSURE_SENSOR_SIG: track 37.1 -> 27.1 mm
- net /AC_RELAYS: track 17.7 -> 9.72 mm
- net /BOILER_TRIAC: track 45.2 -> 40.4 mm
- net Net-(Q3-G): track 90.8 -> 92.6 mm
- net /STEAM_VALVE_IN: track 45.1 -> 43.5 mm, vias 1 -> 0
- added copper zone on B.Cu, net 120VAC_HOT
Other:
- board text added: "+5V"
- board text added: "120VAC"
- board text added: "5VDC"
- board text added: "Boiler Triac In"
- board text added: "Espresso Machine Controller Project"
- board text added: "GND"
- board text added: "NC"
- board text added: "Power Control Board"
- board text added: "Pres. Sensor Out"
- board text added: "Pump Triac In"
- board text added: "Relay In"
- board text added: "Stm Out"
- board text added: "ZC Out"
- board text removed: "120VAC HV"
- board text removed: "5VDC LV"
- board text removed: "HV 120VAC"

Commit message: Boards finalized and ordered
Parts:
- removed R18: 10k, Resistor_SMD:R_0603_1608Metric_Pad0.98x0.95mm_HandSolder
- removed R19: 20k, Resistor_SMD:R_0603_1608Metric_Pad0.98x0.95mm_HandSolder
- U4: renamed from ACDC Converter
Routing:
- net /STEAM_VALVE_IN: track 43.5 -> 36.1 mm
